File: NerdNOS.kicad_pcb (KiCad board)
At the start: 2 copper layers, 60.6 x 25.5 mm, 53 parts, among them IC1 BM1397_mode1, J3 USB_C_Receptacle_USB2.0, Q1 2N7002, U1 T-Display-S3, U2 25MHz, U3 MCP1824T-1802E, U4 MCP1824T-0802E, U6 TXU0202DCUR, U7 TPS566247DRLR

Commit message: BM1366
BM1366 tryout
Parts:
- removed C1: 0.1uF, Capacitor_SMD:C_0402_1005Metric
- removed C12, C14, C15, C16, C17, C18, C2, C3, C4, C5, C6, C8: 1uF, Capacitor_SMD:C_0402_1005Metric
- removed IC1: BM1397_mode1, bitaxe:BM1397
- removed Q1: 2N7002, Package_TO_SOT_SMD:SOT-23
- removed R14, R5: 10k, Resistor_SMD:R_0402_1005Metric
- removed R2: 1k, Resistor_SMD:R_0402_1005Metric
- removed U2: 25MHz, bitaxe:O 25,0-JO32-B-1V3-1-T1-LF
- added C10: 1uF, Capacitor_SMD:C_0402_1005Metric, F.Cu at (107.5, 61.2)
- added C23: 1uF, Capacitor_SMD:C_0402_1005Metric, F.Cu at (108.5, 61.2)
- added C24: 1uF, Capacitor_SMD:C_0402_1005Metric, F.Cu at (109.6, 61.3)
- added C27: 1uF, Capacitor_SMD:C_0402_1005Metric, F.Cu at (108.9, 63.2)
- added C28: 1uF, Capacitor_SMD:C_0402_1005Metric, F.Cu at (108.9, 69.3)
- added C31: 1uF, Capacitor_SMD:C_0402_1005Metric, F.Cu at (109.2, 71.3)
- added C32: 1uF, Capacitor_SMD:C_0402_1005Metric, F.Cu at (108.0, 71.2)
- added C33: 1uF, Capacitor_SMD:C_0402_1005Metric, F.Cu at (107.0, 71.1)
- added C34: 1uF, Capacitor_SMD:C_0402_1005Metric, F.Cu at (102.3, 71.0)
- added C35: 1uF, Capacitor_SMD:C_0402_1005Metric, F.Cu at (101.4, 70.9)
- added C36: 1uF, Capacitor_SMD:C_0402_1005Metric, F.Cu at (101.4, 61.4)
- added C37: 1uF, Capacitor_SMD:C_0402_1005Metric, F.Cu at (102.4, 61.4)
- added C38: 0.1uF, Capacitor_SMD:C_0402_1005Metric, F.Cu at (93.1, 67.5)
- added Q2: 2N7002, Package_TO_SOT_SMD:SOT-23, F.Cu at (84.9, 67.5)
- added R3: 10k, Resistor_SMD:R_0402_1005Metric, F.Cu at (104.7, 71.2)
- added R4: 10k, Resistor_SMD:R_0402_1005Metric, F.Cu at (85.1, 70.0)
- added R9: 5.1k, Resistor_SMD:R_0402_1005Metric, F.Cu at (85.8, 65.0)
- added U5: BM1366_mode1, bitaxe:BM1366, F.Cu at (104.3, 66.3)
- added U8: 25MHz, bitaxe:O 25,0-JO32-B-1V3-1-T1-LF, F.Cu at (91.7, 65.2)
- R1: value 5.1k -> 10k; footprint Resistor_SMD:R_0402_1005Metric -> PCM_Resistor_SMD_AKL:R_0402_1005Metric
- R12: value 13.3k -> 9.31k
- moved R1 19.9 mm to (105.4, 61.2), turned to -90 degrees
- moved G*** 1.17 mm to (133.3, 75.7)
- moved TH1 0.29 mm to (100.0, 66.2)
Connections:
- R1 pad 1: /BM1397/RST_N -> GND
- R1 pad 2: /BM1397/1V8 -> Net-(U5-BI)
Routing:
- net GND: track 48.5 -> 53.4 mm, vias 76 -> 61
- net Net-(U5-VDD2_0): track 0.00 -> 4.02 mm
- net Net-(U5-VDD3_0): track 0.00 -> 3.52 mm
- net /BM1397/VDD: track 40.6 -> 44.1 mm, vias 0 -> 8
- net Net-(U5-VDD2_1): track 0.00 -> 3.45 mm
- net Net-(IC1-VDD2_0): track 3.34 -> 0.00 mm
- net Net-(IC1-VDD2_1): track 3.32 -> 0.00 mm
- net /BM1397/1V8: track 50.9 -> 54.2 mm
- net Net-(IC1-VDD3_0): track 3.22 -> 0.00 mm
- net Net-(IC1-VDD1_0): track 3.22 -> 0.00 mm
- net Net-(IC1-VDD1_1): track 3.20 -> 0.00 mm
- net Net-(IC1-VDD3_1): track 3.15 -> 0.00 mm
- net Net-(U5-VDD1_0): track 0.00 -> 3.11 mm
- net Net-(U5-VDD3_1): track 0.00 -> 3.10 mm
- net Net-(U5-VDD1_1): track 0.00 -> 2.77 mm
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Other:
- board text added: "Ultra"
- board text removed: "1.3"
