File: power.kicad_sch (KiCad schematic)
At the start: 10 parts, among them U7 TPS566247DRLR

Commit message: BM1366
BM1366 tryout
Parts:
- R12: value 13.3k -> 10k
Changed lines of the file:
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@@
 			)
 		)
-		(property "Value" "13.3k"
+		(property "Value" "10k"
 			(at 160.655 73.025 90)
 			(effects
